Commit message: Added inertia

File: fl_description/urdf/fanuc_macro.xacro (robot description, xacro)
@@ -18,4 +18,8 @@
         </geometry>
       </collision>
+      <inertial>
+        <mass value="200"/>
+        <inertia ixx="0" ixy="0" ixz="0" iyy="0" iyz="0" izz="0"/>
+      </inertial>
     </link>
     <link name="${prefix}link_1">
@@ -33,4 +37,8 @@
         </geometry>
       </collision>
+      <inertial>
+        <mass value="15"/>
+        <inertia ixx="0" ixy="0" ixz="0" iyy="0" iyz="0" izz="0"/>
+      </inertial>
     </link>
     <link name="${prefix}link_2">
@@ -48,4 +56,8 @@
         </geometry>
       </collision>
+      <inertial>
+        <mass value="7"/>
+        <inertia ixx="0" ixy="0" ixz="0" iyy="0" iyz="0" izz="0"/>
+      </inertial>
     </link>
     <link name="${prefix}link_3">
@@ -63,4 +75,8 @@
         </geometry>
       </collision>
+      <inertial>
+        <mass value="4"/>
+        <inertia ixx="0" ixy="0" ixz="0" iyy="0" iyz="0" izz="0"/>
+      </inertial>
     </link>
     <link name="${prefix}link_4">
@@ -78,4 +94,8 @@
         </geometry>
       </collision>
+      <inertial>
+        <mass value="4"/>
+        <inertia ixx="0.47" ixy="0" ixz="0" iyy="0" iyz="0" izz="0"/>
+      </inertial>
     </link>
     <link name="${prefix}link_5">
@@ -93,4 +113,8 @@
         </geometry>
       </collision>
+      <inertial>
+        <mass value="1"/>
+        <inertia ixx="0" ixy="0" ixz="0" iyy="0.47" iyz="0" izz="0"/>
+      </inertial>
     </link>
     <link name="${prefix}link_6">
@@ -108,4 +132,8 @@
         </geometry>
       </collision>
+      <inertial>
+        <mass value="1"/>
+        <inertia ixx="0.15" ixy="0" ixz="0" iyy="0" iyz="0" izz="0"/>
+      </inertial>
     </link>
     <!-- joints: main serial chain -->
