Commit message: Added colors & small refactoring

File: fl_description/urdf/fanuc.xacro (robot description, xacro)
@@ -1,4 +1,4 @@
 <?xml version="1.0" ?>
-<robot name="fanuc" xmlns:xacro="http://ros.org/wiki/xacro">
+<robot name="fanuc_cr7ial" xmlns:xacro="http://ros.org/wiki/xacro">
   <xacro:include filename="$(find fl_description)/urdf/fanuc_macro.xacro"/>
   <fanuc_cr7ial prefix=""/>

File: fl_description/urdf/fanuc_macro.xacro (robot description, xacro)
@@ -1,5 +1,4 @@
 <?xml version="1.0" ?>
 <robot xmlns:xacro="http://ros.org/wiki/xacro">
-	<xacro:include filename="$(find fl_description)/resources/common_materials.xacro"/>
   <xacro:macro name="fanuc_cr7ial" params="prefix">
     <!-- links: main serial chain -->
@@ -10,7 +9,4 @@
           <mesh filename="package://fl_description/meshes/cr7ia/visual/base_link.stl"/>
         </geometry>
-        <material name="">
-      <color rgba="${0/255} ${155/255} ${ 70/255} 1.0"/>
-    </material>
       </visual>
       <collision>
@@ -34,5 +30,4 @@
           <mesh filename="package://fl_description/meshes/cr7ia/visual/link_1.stl"/>
         </geometry>
-        <xacro:material_fanuc_green />
       </visual>
       <collision>
@@ -56,5 +51,4 @@
           <mesh filename="package://fl_description/meshes/cr7ial/visual/link_2.stl"/>
         </geometry>
-        <xacro:material_fanuc_green />
       </visual>
       <collision>
@@ -78,5 +72,4 @@
           <mesh filename="package://fl_description/meshes/cr7ia/visual/link_3.stl"/>
         </geometry>
-        <xacro:material_fanuc_green />
       </visual>
       <collision>
@@ -100,5 +93,4 @@
           <mesh filename="package://fl_description/meshes/cr7ial/visual/link_4.stl"/>
         </geometry>
-        <xacro:material_fanuc_green />
       </visual>
       <collision>
@@ -122,5 +114,4 @@
           <mesh filename="package://fl_description/meshes/cr7ia/visual/link_5.stl"/>
         </geometry>
-        <xacro:material_fanuc_green />
       </visual>
       <collision>
@@ -144,5 +135,4 @@
           <mesh filename="package://fl_description/meshes/cr7ia/visual/link_6.stl"/>
         </geometry>
-        <xacro:material_fanuc_gray24 />
       </visual>
       <collision>
@@ -224,4 +214,25 @@
       <child link="${prefix}tool0" />
     </joint>
+    <gazebo reference="base_link">
+    <material>Gazebo/Green</material>
+    </gazebo>
+    <gazebo reference="link_1">
+    <material>Gazebo/Gray</material>
+    </gazebo>
+    <gazebo reference="link_2">
+    <material>Gazebo/Green</material>
+    </gazebo>
+    <gazebo reference="link_3">
+    <material>Gazebo/Gray</material>
+    </gazebo>
+    <gazebo reference="link_4">
+    <material>Gazebo/Green</material>
+    </gazebo>
+    <gazebo reference="link_5">
+    <material>Gazebo/Gray</material>
+    </gazebo>
+    <gazebo reference="link_6">
+    <material>Gazebo/Black</material>
+    </gazebo>
   </xacro:macro>
 </robot>

Commit message: joint trajectory control done

File: fl_description/urdf/fanuc.xacro (robot description, xacro)
@@ -1,5 +1,15 @@
 <?xml version="1.0" ?>
 <robot name="fanuc_cr7ial" xmlns:xacro="http://ros.org/wiki/xacro">
+	<gazebo>
+    <plugin name="ros_control" filename="libgazebo_ros_control.so">
+    </plugin>
+  </gazebo>
   <xacro:include filename="$(find fl_description)/urdf/fanuc_macro.xacro"/>
   <fanuc_cr7ial prefix=""/>
+  <link name="world" />
+  <joint name="world_joint" type="fixed">
+    <parent link="world" />
+    <child link = "base_link" />
+    <origin xyz="0.0 0.0 0.0" rpy="0.0 0.0 0.0" />
+  </joint>
 </robot>

File: fl_description/urdf/fanuc_macro.xacro (robot description, xacro)
@@ -1,4 +1,15 @@
 <?xml version="1.0" ?>
 <robot xmlns:xacro="http://ros.org/wiki/xacro">
+  <xacro:macro name="joint_transmission_macro" params="joint_name">
+    <transmission name="${joint_name}_transmssion">
+      <type>transmission_interface/SimpleTransmission</type>
+      <joint name="${joint_name}">
+        <hardwareInterface>hardware_interface/PositionJointInterface</hardwareInterface>
+      </joint>
+      <actuator name="${joint_name}_motor">
+        <mechanicalReduction>1</mechanicalReduction>
+      </actuator>
+    </transmission>
+  </xacro:macro>
   <xacro:macro name="fanuc_cr7ial" params="prefix">
     <!-- links: main serial chain -->
@@ -214,4 +225,10 @@
       <child link="${prefix}tool0" />
     </joint>
+  <joint_transmission_macro joint_name="${prefix}joint_1"/>
+  <joint_transmission_macro joint_name="${prefix}joint_2"/>
+  <joint_transmission_macro joint_name="${prefix}joint_3"/>
+  <joint_transmission_macro joint_name="${prefix}joint_4"/>
+  <joint_transmission_macro joint_name="${prefix}joint_5"/>
+  <joint_transmission_macro joint_name="${prefix}joint_6"/>
     <gazebo reference="base_link">
     <material>Gazebo/Green</material>

Commit message: camera and table added

File: fl_description/urdf/fanuc.xacro (robot description, xacro)
@@ -1,15 +1,20 @@
 <?xml version="1.0" ?>
 <robot name="fanuc_cr7ial" xmlns:xacro="http://ros.org/wiki/xacro">
-	<gazebo>
-    <plugin name="ros_control" filename="libgazebo_ros_control.so">
-    </plugin>
-  </gazebo>
-  <xacro:include filename="$(find fl_description)/urdf/fanuc_macro.xacro"/>
-  <fanuc_cr7ial prefix=""/>
-  <link name="world" />
-  <joint name="world_joint" type="fixed">
-    <parent link="world" />
-    <child link = "base_link" />
-    <origin xyz="0.0 0.0 0.0" rpy="0.0 0.0 0.0" />
-  </joint>
+    <gazebo>
+        <plugin name="ros_control" filename="libgazebo_ros_control.so">
+        </plugin>
+    </gazebo>
+    <link name="world"/>
+    <xacro:include filename="$(find fl_description)/urdf/fanuc_macro.xacro"/>
+    <fanuc_cr7ial prefix="" parent="world"/>
+    <xacro:include filename="$(find fl_description)/urdf/camera.urdf.xacro"/>
+    <camera_sensor xyz="0.5 0 2"
+                   rpy="0 ${3.1415/2} 0" parent="world"
+                   name="camera" topic="fl_camera">
+    </camera_sensor>
+    <xacro:include filename="$(find fl_description)/urdf/table.urdf.xacro"/>
+    <table_macro xyz="0.5 0 0"
+                 size="1 2 0.4" parent="world"
+                 color="color_camera" name="fl_table">
+    </table_macro>
 </robot>

File: fl_description/urdf/fanuc_macro.xacro (robot description, xacro)
@@ -12,5 +12,10 @@
     </transmission>
   </xacro:macro>
-  <xacro:macro name="fanuc_cr7ial" params="prefix">
+  <xacro:macro name="fanuc_cr7ial" params="prefix parent">
+      <joint name="world_joint" type="fixed">
+    <parent link="${parent}" />
+    <child link = "${prefix}base_link" />
+    <origin xyz="0.0 0.0 0.0" rpy="0.0 0.0 0.0" />
+  </joint>
     <!-- links: main serial chain -->
     <link name="${prefix}base_link">
