Commit message: Added decorative changes in simulator & fixed errors in control

File: fl_description/urdf/brick.xacro (robot description, xacro)
@@ -2,5 +2,5 @@
 <robot xmlns:xacro="http://www.ros.org/wiki/xacro" name="camera">
     <xacro:include filename="$(find fl_description)/urdf/parameters.xacro"/>
-    <xacro:macro name="table_macro" params="xyz color parent name size">
+    <xacro:macro name="brick_macro" params="xyz color parent name size">
         <joint name="${name}_joint" type="fixed">
             <axis xyz="0 1 0"/>
@@ -31,5 +31,5 @@
         </link>
         <gazebo reference="${name}">
-            <material>Gazebo/White</material>
+            <material>Gazebo/Red</material>
         </gazebo>
     </xacro:macro>

File: fl_description/urdf/camera.urdf.xacro (robot description, xacro)
@@ -32,11 +32,11 @@
             <material>Gazebo/Yellow</material>
             <sensor type="camera" name="${name}_sensor">
-                <update_rate>30.0</update_rate>
+                <update_rate>5.0</update_rate>
                 <camera name="head">
                     <horizontal_fov>1.3962634</horizontal_fov>
                     <image>
-                        <width>800</width>
-                        <height>800</height>
-                        <format>R8G8B8</format>
+                        <width>1200</width>
+                        <height>1200</height>
+                        <format>B8G8R8</format>
                     </image>
                     <clip>

File: fl_description/urdf/fanuc.xacro (robot description, xacro)
@@ -9,5 +9,5 @@
     <fanuc_cr7ial prefix="" parent="world"/>
     <xacro:include filename="$(find fl_description)/urdf/camera.urdf.xacro"/>
-    <camera_sensor xyz="0.5 0 2"
+    <camera_sensor xyz="0.5 0 1.45"
                    rpy="0 ${3.1415/2} 0" parent="world"
                    name="camera" topic="fl_camera">
@@ -15,6 +15,17 @@
     <xacro:include filename="$(find fl_description)/urdf/table.urdf.xacro"/>
     <table_macro xyz="0.5 0 0"
-                 size="1 2 0.4" parent="world"
-                 color="color_camera" name="fl_table">
+                 size="1.2 1.2 0.6" parent="world"
+                 color="white" name="fl_table">
     </table_macro>
+    <xacro:include filename="$(find fl_description)/urdf/brick.xacro"/>
+    <table_macro xyz="0.5 0.2 0.35"
+                 size="0.1 0.1 0.1" parent="world"
+                 color="red" name="fl_box">
+    </table_macro>
+        <gazebo reference="fl_box">
+            <material>Gazebo/Orange</material>
+        </gazebo>
+        <gazebo reference="fl_table">
+            <material>Gazebo/White</material>
+        </gazebo>
 </robot>

File: fl_description/urdf/fanuc_macro.xacro (robot description, xacro)
@@ -240,5 +240,5 @@
     </gazebo>
     <gazebo reference="link_1">
-    <material>Gazebo/Gray</material>
+    <material>Gazebo/Green</material>
     </gazebo>
     <gazebo reference="link_2">
@@ -246,5 +246,5 @@
     </gazebo>
     <gazebo reference="link_3">
-    <material>Gazebo/Gray</material>
+    <material>Gazebo/Green</material>
     </gazebo>
     <gazebo reference="link_4">
@@ -252,8 +252,8 @@
     </gazebo>
     <gazebo reference="link_5">
-    <material>Gazebo/Gray</material>
+    <material>Gazebo/Green</material>
     </gazebo>
     <gazebo reference="link_6">
-    <material>Gazebo/Black</material>
+    <material>Gazebo/Green</material>
     </gazebo>
   </xacro:macro>

Commit message: small refactoring

File: fl_description/urdf/brick.xacro (robot description, xacro)
@@ -1,6 +1,6 @@
 <?xml version="1.0"?>
-<robot xmlns:xacro="http://www.ros.org/wiki/xacro" name="camera">
+<robot xmlns:xacro="http://www.ros.org/wiki/xacro">
     <xacro:include filename="$(find fl_description)/urdf/parameters.xacro"/>
-    <xacro:macro name="brick_macro" params="xyz color parent name size">
+    <xacro:macro name="brick_macro" params="xyz parent name size">
         <joint name="${name}_joint" type="fixed">
             <axis xyz="0 1 0"/>
@@ -21,5 +21,4 @@
                     <box size="${size}"/>
                 </geometry>
-                <material name="${color}"/>
             </visual>
             <inertial>

File: fl_description/urdf/camera.urdf.xacro (robot description, xacro)
@@ -1,4 +1,4 @@
 <?xml version="1.0"?>
-<robot xmlns:xacro="http://www.ros.org/wiki/xacro" name="camera">
+<robot xmlns:xacro="http://www.ros.org/wiki/xacro" >
     <xacro:include filename="$(find fl_description)/urdf/parameters.xacro"/>
     <xacro:macro name="camera_sensor" params="xyz rpy parent name topic">

File: fl_description/urdf/fanuc.xacro (robot description, xacro)
@@ -1,4 +1,4 @@
 <?xml version="1.0" ?>
-<robot name="fanuc_cr7ial" xmlns:xacro="http://ros.org/wiki/xacro">
+<robot name="fanuc_cr7ial" xmlns:xacro="http://www.ros.org/wiki/xacro">
     <gazebo>
         <plugin name="ros_control" filename="libgazebo_ros_control.so">
@@ -11,21 +11,15 @@
     <camera_sensor xyz="0.5 0 1.45"
                    rpy="0 ${3.1415/2} 0" parent="world"
-                   name="camera" topic="fl_camera">
+                   name="camera" topic="fanlearn_camera">
     </camera_sensor>
     <xacro:include filename="$(find fl_description)/urdf/table.urdf.xacro"/>
     <table_macro xyz="0.5 0 0"
                  size="1.2 1.2 0.6" parent="world"
-                 color="white" name="fl_table">
+                 name="fl_table">
     </table_macro>
     <xacro:include filename="$(find fl_description)/urdf/brick.xacro"/>
-    <table_macro xyz="0.5 0.2 0.35"
+    <brick_macro xyz="0.5 0.2 0.35"
                  size="0.1 0.1 0.1" parent="world"
-                 color="red" name="fl_box">
-    </table_macro>
-        <gazebo reference="fl_box">
-            <material>Gazebo/Orange</material>
-        </gazebo>
-        <gazebo reference="fl_table">
-            <material>Gazebo/White</material>
-        </gazebo>
+                 name="fl_box">
+    </brick_macro>
 </robot>

File: fl_description/urdf/fanuc_macro.xacro (robot description, xacro)
@@ -1,4 +1,4 @@
 <?xml version="1.0" ?>
-<robot xmlns:xacro="http://ros.org/wiki/xacro">
+<robot xmlns:xacro="http://www.ros.org/wiki/xacro">
   <xacro:macro name="joint_transmission_macro" params="joint_name">
     <transmission name="${joint_name}_transmssion">

File: fl_description/urdf/parameters.xacro (robot description, xacro)
@@ -1,4 +1,4 @@
 <?xml version="1.0" encoding="UTF-8"?>
-<robot xmlns:xacro="http://www.ros.org/wiki/xacro" name="plato_robot">
+<robot xmlns:xacro="http://www.ros.org/wiki/xacro">
     <!-- Camera properties -->
     <xacro:property name="camera_size" value="0.02"/>

File: fl_description/urdf/table.urdf.xacro (robot description, xacro)
@@ -1,6 +1,6 @@
 <?xml version="1.0"?>
-<robot xmlns:xacro="http://www.ros.org/wiki/xacro" name="camera">
+<robot xmlns:xacro="http://www.ros.org/wiki/xacro" >
     <xacro:include filename="$(find fl_description)/urdf/parameters.xacro"/>
-    <xacro:macro name="table_macro" params="xyz color parent name size">
+    <xacro:macro name="table_macro" params="xyz parent name size">
         <joint name="${name}_joint" type="fixed">
             <axis xyz="0 1 0"/>
@@ -21,5 +21,4 @@
                     <box size="${size}"/>
                 </geometry>
-                <material name="${color}"/>
             </visual>
             <inertial>

Commit message: new coordinates

File: fl_description/urdf/brick.xacro (robot description, xacro)
@@ -23,7 +23,7 @@
             </visual>
             <inertial>
-                <mass value="${table_mass}"/>
+                <mass value="0.1"/>
                 <origin xyz="0 0 0" rpy="0 0 0"/>
-                <box_inertia m="${table_mass}" x="${table_size}" y="${table_size}" z="${table_size}"/>
+                <box_inertia m="0.1" x="${table_size}" y="${table_size}" z="${table_size}"/>
                 <inertia ixx="1e-6" ixy="0" ixz="0" iyy="1e-6" iyz="0" izz="1e-6"/>
             </inertial>

File: fl_description/urdf/fanuc_macro.xacro (robot description, xacro)
@@ -224,5 +224,24 @@
     </joint>
     <!-- ROS-Industrial 'tool0' frame: all-zeros tool frame -->
-    <link name="${prefix}tool0" />
+        <link name="${prefix}tool0" >
+            <collision>
+                <origin xyz="0 0 0" rpy="0 0 0"/>
+                <geometry>
+                    <box size="0.1 0.1 0.1"/>
+                </geometry>
+            </collision>
+            <visual>
+                <origin xyz="0 0 0" rpy="0 0 0"/>
+                <geometry>
+                    <box size="0.1 0.1 0.1"/>
+                </geometry>
+            </visual>
+            <inertial>
+                <mass value="0.1"/>
+                <origin xyz="0 0 0" rpy="0 0 0"/>
+                <box_inertia m="0.1" x="0.1" y="0.1" z="0.1"/>
+                <inertia ixx="1e-6" ixy="0" ixz="0" iyy="1e-6" iyz="0" izz="1e-6"/>
+            </inertial>
+        </link>
     <joint name="${prefix}link_6-tool0" type="fixed">
       <origin xyz="0 0 0" rpy="${pi} ${-pi/2.0} 0" />
@@ -257,4 +276,7 @@
     <material>Gazebo/Green</material>
     </gazebo>
+    <gazebo reference="tool0">
+    <material>Gazebo/Green</material>
+    </gazebo>
   </xacro:macro>
 </robot>

Commit message: Added physics

File: fl_description/urdf/brick.xacro (robot description, xacro)
@@ -3,9 +3,10 @@
     <xacro:include filename="$(find fl_description)/urdf/parameters.xacro"/>
     <xacro:macro name="brick_macro" params="xyz parent name size">
-        <joint name="${name}_joint" type="fixed">
+        <joint name="${name}_joint" type="floating">
             <axis xyz="0 1 0"/>
             <origin xyz="${xyz}" rpy="0 0 0"/>
             <parent link="${parent}"/>
             <child link="${name}"/>
+            <dynamics damping="7.0" friction="2.0"/>
         </joint>
         <link name="${name}">
@@ -15,4 +16,13 @@
                     <box size="${size}"/>
                 </geometry>
+                <surface>
+                    <friction>
+                        <ode mu="10.0" mu2="10.0" fdir1="1 1 1" slip1="1" slip2="1"/>
+                    </friction>
+                    <bounce restitution_coefficient="1" threshold="1000000.0"/>
+                    <contact>
+                        <ode soft_cfm="1" soft_erp="0.2" kp="1e10" kd="1.0" max_vel="1.0" min_depth="0.0001"/>
+                    </contact>
+                </surface>
             </collision>
             <visual>
@@ -26,9 +36,13 @@
                 <origin xyz="0 0 0" rpy="0 0 0"/>
                 <box_inertia m="0.1" x="${table_size}" y="${table_size}" z="${table_size}"/>
-                <inertia ixx="1e-6" ixy="0" ixz="0" iyy="1e-6" iyz="0" izz="1e-6"/>
+                <inertia ixx="1.0" ixy="1.0" ixz="1.0" iyy="1.0" iyz="1.0" izz="1.0"/>
             </inertial>
         </link>
         <gazebo reference="${name}">
+            <turnGravityOff>false</turnGravityOff>
             <material>Gazebo/Red</material>
+                <mu1>1</mu1>
+            <mu2>1</mu2>
+            <selfCollide>true</selfCollide>
         </gazebo>
     </xacro:macro>

File: fl_description/urdf/fanuc_macro.xacro (robot description, xacro)
@@ -274,5 +274,8 @@
     </gazebo>
     <gazebo reference="link_6">
-    <material>Gazebo/Green</material>
+      <material>Gazebo/Green</material>
+      <mu1>1</mu1>
+        <mu2>1</mu2>
+    <selfCollide>true</selfCollide>
     </gazebo>
     <gazebo reference="tool0">

File: fl_description/urdf/table.urdf.xacro (robot description, xacro)
@@ -8,4 +8,5 @@
             <parent link="${parent}"/>
             <child link="${name}"/>
+            <dynamics damping="7.0" friction="2.0"/>
         </joint>
         <link name="${name}">
@@ -15,4 +16,13 @@
                     <box size="${size}"/>
                 </geometry>
+                <surface>
+                    <friction>
+                        <ode mu="10.0" mu2="10.0" fdir1="1 1 1" slip1="1" slip2="1"/>
+                    </friction>
+                    <bounce restitution_coefficient="1" threshold="1000000.0"/>
+                    <contact>
+                        <ode soft_cfm="1" soft_erp="0.2" kp="1e10" kd="1" max_vel="100.0" min_depth="0.0001"/>
+                    </contact>
+                </surface>
             </collision>
             <visual>
@@ -26,9 +36,12 @@
                 <origin xyz="0 0 0" rpy="0 0 0"/>
                 <box_inertia m="${table_mass}" x="${table_size}" y="${table_size}" z="${table_size}"/>
-                <inertia ixx="1e-6" ixy="0" ixz="0" iyy="1e-6" iyz="0" izz="1e-6"/>
+                <inertia ixx="1.0" ixy="1.0" ixz="1.0" iyy="1.0" iyz="1.0" izz="1.0"/>
             </inertial>
         </link>
         <gazebo reference="${name}">
             <material>Gazebo/White</material>
+                <mu1>1</mu1>
+            <mu2>1</mu2>
+            <selfCollide>true</selfCollide>
         </gazebo>
     </xacro:macro>
