Commit message: Added generated files from moveit

File: fl_description/resources/common_colours.xacro (robot description, xacro)
@@ -1,4 +1,4 @@
 <?xml version="1.0"?>
-<robot xmlns:xacro="http://wiki.ros.org/xacro">
+<robot xmlns:xacro="http://ros.org/wiki/xacro">
   <!-- RAL 1021: Rape yellow -->
   <xacro:property name="color_fanuc_yellow"   value="0.96 0.76 0.13 1.0" />

File: fl_description/resources/common_materials.xacro (robot description, xacro)
@@ -1,4 +1,4 @@
 <?xml version="1.0"?>
-<robot xmlns:xacro="http://wiki.ros.org/xacro">
+<robot xmlns:xacro="http://ros.org/wiki/xacro">
   <xacro:include filename="$(find fl_description)/resources/common_colours.xacro"/>
   <xacro:macro name="material_fanuc_yellow">

File: fl_description/urdf/fanuc.xacro (robot description, xacro)
@@ -1,4 +1,4 @@
 <?xml version="1.0" ?>
-<robot name="fanuc_cr7ial" xmlns:xacro="http://ros.org/wiki/xacro">
+<robot name="fanuc" xmlns:xacro="http://ros.org/wiki/xacro">
   <xacro:include filename="$(find fl_description)/urdf/fanuc_macro.xacro"/>
   <fanuc_cr7ial prefix=""/>

File: fl_description/urdf/fanuc_macro.xacro (robot description, xacro)
@@ -10,4 +10,138 @@
           <mesh filename="package://fl_description/meshes/cr7ia/visual/base_link.stl"/>
         </geometry>
+        <material name="">
+      <color rgba="${0/255} ${155/255} ${ 70/255} 1.0"/>
+    </material>
+      </visual>
+      <collision>
+        <origin xyz="0 0 0" rpy="0 0 0"/>
+        <geometry>
+          <mesh filename="package://fl_description/meshes/cr7ia/collision/base_link.stl"/>
+        </geometry>
+      </collision>
+      <inertial>
+        <mass value="100"/>
+        <inertia
+          ixx="0" ixy="0" ixz="0"
+          iyy="0" iyz="0"
+          izz="0"/>
+      </inertial>
+    </link>
+    <link name="${prefix}link_1">
+      <visual>
+        <origin xyz="0 0 0" rpy="0 0 0"/>
+        <geometry>
+          <mesh filename="package://fl_description/meshes/cr7ia/visual/link_1.stl"/>
+        </geometry>
+        <xacro:material_fanuc_green />
+      </visual>
+      <collision>
+        <origin xyz="0 0 0" rpy="0 0 0"/>
+        <geometry>
+          <mesh filename="package://fl_description/meshes/cr7ia/collision/link_1.stl"/>
+        </geometry>
+      </collision>
+      <inertial>
+        <mass value="15"/>
+        <inertia
+          ixx="0" ixy="0" ixz="0"
+          iyy="0" iyz="0"
+          izz="0"/>
+      </inertial>
+    </link>
+    <link name="${prefix}link_2">
+      <visual>
+        <origin xyz="0 0 0" rpy="0 0 0"/>
+        <geometry>
+          <mesh filename="package://fl_description/meshes/cr7ial/visual/link_2.stl"/>
+        </geometry>
+        <xacro:material_fanuc_green />
+      </visual>
+      <collision>
+        <origin xyz="0 0 0" rpy="0 0 0"/>
+        <geometry>
+          <mesh filename="package://fl_description/meshes/cr7ial/collision/link_2.stl"/>
+        </geometry>
+      </collision>
+      <inertial>
+        <mass value="7"/>
+        <inertia
+          ixx="0" ixy="0" ixz="0"
+          iyy="0" iyz="0"
+          izz="0"/>
+      </inertial>
+    </link>
+    <link name="${prefix}link_3">
+      <visual>
+        <origin xyz="0 0 0" rpy="0 0 0"/>
+        <geometry>
+          <mesh filename="package://fl_description/meshes/cr7ia/visual/link_3.stl"/>
+        </geometry>
+        <xacro:material_fanuc_green />
+      </visual>
+      <collision>
+        <origin xyz="0 0 0" rpy="0 0 0"/>
+        <geometry>
+          <mesh filename="package://fl_description/meshes/cr7ia/collision/link_3.stl"/>
+        </geometry>
+      </collision>
+      <inertial>
+        <mass value="4"/>
+        <inertia
+          ixx="0" ixy="0" ixz="0"
+          iyy="0" iyz="0"
+          izz="0"/>
+      </inertial>
+    </link>
+    <link name="${prefix}link_4">
+      <visual>
+        <origin xyz="0 0 0" rpy="0 0 0"/>
+        <geometry>
+          <mesh filename="package://fl_description/meshes/cr7ial/visual/link_4.stl"/>
+        </geometry>
+        <xacro:material_fanuc_green />
+      </visual>
+      <collision>
+        <origin xyz="0 0 0" rpy="0 0 0"/>
+        <geometry>
+          <mesh filename="package://fl_description/meshes/cr7ial/collision/link_4.stl"/>
+        </geometry>
+      </collision>
+      <inertial>
+        <mass value="4"/>
+        <inertia
+          ixx="0.47" ixy="0" ixz="0"
+          iyy="0" iyz="0"
+          izz="0"/>
+      </inertial>
+    </link>
+    <link name="${prefix}link_5">
+      <visual>
+        <origin xyz="0 0 0" rpy="0 0 0"/>
+        <geometry>
+          <mesh filename="package://fl_description/meshes/cr7ia/visual/link_5.stl"/>
+        </geometry>
+        <xacro:material_fanuc_green />
+      </visual>
+      <collision>
+        <origin xyz="0 0 0" rpy="0 0 0"/>
+        <geometry>
+          <mesh filename="package://fl_description/meshes/cr7ia/collision/link_5.stl"/>
+        </geometry>
+      </collision>
+      <inertial>
+        <mass value="1"/>
+        <inertia
+          ixx="0" ixy="0" ixz="0"
+          iyy="0.47" iyz="0"
+          izz="0"/>
+      </inertial>
+    </link>
+    <link name="${prefix}link_6">
+      <visual>
+        <origin xyz="0 0 0" rpy="0 0 0"/>
+        <geometry>
+          <mesh filename="package://fl_description/meshes/cr7ia/visual/link_6.stl"/>
+        </geometry>
         <xacro:material_fanuc_gray24 />
       </visual>
@@ -15,124 +149,13 @@
         <origin xyz="0 0 0" rpy="0 0 0"/>
         <geometry>
-          <mesh filename="package://fl_description/meshes/cr7ia/collision/base_link.stl"/>
-        </geometry>
-      </collision>
-      <inertial>
-        <mass value="200"/>
-        <inertia ixx="0" ixy="0" ixz="0" iyy="0" iyz="0" izz="0"/>
-      </inertial>
-    </link>
-    <link name="${prefix}link_1">
-      <visual>
-        <origin xyz="0 0 0" rpy="0 0 0"/>
-        <geometry>
-          <mesh filename="package://fl_description/meshes/cr7ia/visual/link_1.stl"/>
-        </geometry>
-        <xacro:material_fanuc_green />
-      </visual>
-      <collision>
-        <origin xyz="0 0 0" rpy="0 0 0"/>
-        <geometry>
-          <mesh filename="package://fl_description/meshes/cr7ia/collision/link_1.stl"/>
-        </geometry>
-      </collision>
-      <inertial>
-        <mass value="15"/>
-        <inertia ixx="0" ixy="0" ixz="0" iyy="0" iyz="0" izz="0"/>
-      </inertial>
-    </link>
-    <link name="${prefix}link_2">
-      <visual>
-        <origin xyz="0 0 0" rpy="0 0 0"/>
-        <geometry>
-          <mesh filename="package://fl_description/meshes/cr7ial/visual/link_2.stl"/>
-        </geometry>
-        <xacro:material_fanuc_green />
-      </visual>
-      <collision>
-        <origin xyz="0 0 0" rpy="0 0 0"/>
-        <geometry>
-          <mesh filename="package://fl_description/meshes/cr7ial/collision/link_2.stl"/>
-        </geometry>
-      </collision>
-      <inertial>
-        <mass value="7"/>
-        <inertia ixx="0" ixy="0" ixz="0" iyy="0" iyz="0" izz="0"/>
-      </inertial>
-    </link>
-    <link name="${prefix}link_3">
-      <visual>
-        <origin xyz="0 0 0" rpy="0 0 0"/>
-        <geometry>
-          <mesh filename="package://fl_description/meshes/cr7ia/visual/link_3.stl"/>
-        </geometry>
-        <xacro:material_fanuc_green />
-      </visual>
-      <collision>
-        <origin xyz="0 0 0" rpy="0 0 0"/>
-        <geometry>
-          <mesh filename="package://fl_description/meshes/cr7ia/collision/link_3.stl"/>
-        </geometry>
-      </collision>
-      <inertial>
-        <mass value="4"/>
-        <inertia ixx="0" ixy="0" ixz="0" iyy="0" iyz="0" izz="0"/>
-      </inertial>
-    </link>
-    <link name="${prefix}link_4">
-      <visual>
-        <origin xyz="0 0 0" rpy="0 0 0"/>
-        <geometry>
-          <mesh filename="package://fl_description/meshes/cr7ial/visual/link_4.stl"/>
-        </geometry>
-        <xacro:material_fanuc_green />
-      </visual>
-      <collision>
-        <origin xyz="0 0 0" rpy="0 0 0"/>
-        <geometry>
-          <mesh filename="package://fl_description/meshes/cr7ial/collision/link_4.stl"/>
-        </geometry>
-      </collision>
-      <inertial>
-        <mass value="4"/>
-        <inertia ixx="0.47" ixy="0" ixz="0" iyy="0" iyz="0" izz="0"/>
-      </inertial>
-    </link>
-    <link name="${prefix}link_5">
-      <visual>
-        <origin xyz="0 0 0" rpy="0 0 0"/>
-        <geometry>
-          <mesh filename="package://fl_description/meshes/cr7ia/visual/link_5.stl"/>
-        </geometry>
-        <xacro:material_fanuc_green />
-      </visual>
-      <collision>
-        <origin xyz="0 0 0" rpy="0 0 0"/>
-        <geometry>
-          <mesh filename="package://fl_description/meshes/cr7ia/collision/link_5.stl"/>
+          <mesh filename="package://fl_description/meshes/cr7ia/collision/link_6.stl"/>
         </geometry>
       </collision>
       <inertial>
         <mass value="1"/>
-        <inertia ixx="0" ixy="0" ixz="0" iyy="0.47" iyz="0" izz="0"/>
-      </inertial>
-    </link>
-    <link name="${prefix}link_6">
-      <visual>
-        <origin xyz="0 0 0" rpy="0 0 0"/>
-        <geometry>
-          <mesh filename="package://fl_description/meshes/cr7ia/visual/link_6.stl"/>
-        </geometry>
-        <xacro:material_fanuc_gray24 />
-      </visual>
-      <collision>
-        <origin xyz="0 0 0" rpy="0 0 0"/>
-        <geometry>
-          <mesh filename="package://fl_description/meshes/cr7ia/collision/link_6.stl"/>
-        </geometry>
-      </collision>
-      <inertial>
-        <mass value="1"/>
-        <inertia ixx="0.15" ixy="0" ixz="0" iyy="0" iyz="0" izz="0"/>
+        <inertia
+          ixx="0.15" ixy="0" ixz="0"
+          iyy="0" iyz="0"
+          izz="0"/>
       </inertial>
     </link>
